File: PCB/PCB/v1.1/MCU.kicad_sch (KiCad schematic)
At the start: 28 parts

Commit message: update PCB file
Parts:
- removed U: (no value), symbol Connector:USB_C_Receptacle_USB2.0
- removed U (x8): (no value), symbol Device:R_Small
- removed U (x2): (no value), symbol Connector_Generic:Conn_01x01
- removed U (x2): (no value), symbol keeb_parts:R_Small
- removed U (x2): (no value), symbol Device:C_Polarized_Small_US
- removed U (x2): (no value), symbol Device:Q_PMOS_GSD
- removed U: (no value), symbol Regulator_Linear:MIC5219-3.3YM5
- removed U (x2): (no value), symbol Device:C
- removed U: E73-2G4M08S1C, symbol kien242:E73-2G4M08S1C
- removed U (x2): (no value), symbol Device:LED
- removed U: (no value), symbol Power_Protection:USBLC6-2SC6
- removed U: (no value), symbol Battery_Management:MCP73831-3-OT
- removed U: (no value), symbol Switch:SW_Push
- removed U: (no value), symbol Device:C_Small
- removed U: (no value), symbol Device:D_Schottky_Small
- added C21, C22: (no value), symbol Device:C_Polarized_Small_US
- added C23: (no value), symbol Device:C_Small
- added C24, C25: (no value), symbol Device:C
- added D43, D45: (no value), symbol Device:LED
- added D44: (no value), symbol Device:D_Schottky_Small
- added J30: USB_C_Receptacle_USB2.0, kien242:USB-C-16pin-hight-v2, symbol Connector:USB_C_Receptacle_USB2.0
- added J31: (no value), kien242:USB-C-16pin-hight-v2, symbol Connector:USB_C_Receptacle_USB2.0
- added J32, J33: (no value), symbol Connector_Generic:Conn_01x01
- added Q1, Q2: (no value), symbol Device:Q_PMOS_GSD
- added R1, R3: (no value), symbol keeb_parts:R_Small
- added R10, R2, R4, R5, R6, R7, R8, R9: (no value), symbol Device:R_Small
- added SW46: (no value), Button_Switch_SMD:SW_SPST_TL3342, symbol Switch:SW_Push
- added U2: (no value), symbol Regulator_Linear:MIC5219-3.3YM5
- added U3: (no value), symbol Power_Protection:USBLC6-2SC6
- added U4: (no value), kien242:E73-2G4M08S1C, symbol kien242:E73-2G4M08S1C
- added U5: (no value), symbol Battery_Management:MCP73831-3-OT
Connections:
- net +3V3: now also C22.1, C24.1, C25.1, Q2.2 (S), U2.5 (OUT)
- net +5V: now also D44.2 (A), D45.2 (A), J30.A4 (VBUS), J30.A9 (VBUS), J30.B4 (VBUS), J30.B9 (VBUS), J31.A4 (VBUS), J31.A9 (VBUS), J31.B4 (VBUS), J31.B9 (VBUS), Q1.1 (G), R7.1, U3.5 (VBUS), U5.4 (VDD)
- net BATTERY_PIN: now also C23.1, R5.2, R8.1
- net D+: now also U3.3 (I/O2)
- net D-: now also U3.1 (I/O1)
- net DP+: now also J30.A6 (D+), J30.B6 (D+), J31.A6 (D+), J31.B6 (D+), U3.4 (I/O2)
- net DP-: now also J30.A7 (D-), J30.B7 (D-), J31.A7 (D-), J31.B7 (D-), U3.6 (I/O1)
- net GND: now also C21.2, C22.2, C23.2, C24.2, C25.2, J30.A1 (GND), J30.A12 (GND), J30.B1 (GND), J30.B12 (GND), J30.S1 (SHIELD), J31.A1 (GND), J31.A12 (GND), J31.B1 (GND), J31.B12 (GND), J31.S1 (SHIELD), R1.2, R10.2, R3.1, R4.1, R6.2, R7.2, R8.2, SW46.1, U2.2 (GND), U3.2 (GND), U5.2 (VSS)
- net LED_1: now also D43.2 (A)
- net POWER_PIN: now also Q2.1 (G), R6.1
- net RST: now also SW46.2
- net SWCLK: now also J32.1 (Pin_1)
- net SWDIO: now also J33.1 (Pin_1)
- net VBAT: now also Q1.3 (D), R2.1, U5.3 (VBAT)
- net VCC: now also Q2.3 (D)
- new net: R10.1, U5.5 (PROG)
- new net: R9.2, U5.1 (STAT)
- new net: R2.2, R5.1
- new net: J30.A5 (CC1), J31.B5 (CC2), R3.2
- new net: J30.B5 (CC2), J31.A5 (CC1), R1.1
- new net: C21.1, D44.1 (K), Q1.2 (S), U2.1 (IN), U2.3 (EN)
- new net: D43.1 (K), R4.2
- new net: D45.1 (K), R9.1

Commit message: update PCB file
Parts:
- C21, C22: value (none) -> 10uF; footprint (none) -> Capacitor_Tantalum_SMD:CP_EIA-3216-12_Kemet-S
- C23, C25: value (none) -> 100nF; footprint (none) -> Capacitor_SMD:C_0603_1608Metric
- C24: value (none) -> 10uF; footprint (none) -> Capacitor_SMD:C_0603_1608Metric
- D43, D45: value (none) -> BLUE; footprint (none) -> LED_SMD:LED_0603_1608Metric
- D44: value (none) -> 1N5819; footprint (none) -> Diode_SMD:D_SOD-323_HandSoldering
- J31: value (none) -> USB_C_Receptacle_USB2.0
- J32: value (none) -> (none); footprint (none) -> TestPoint:TestPoint_Pad_1.5x1.5mm
- J33: value (none) -> (none); footprint (none) -> TestPoint:TestPoint_Pad_D1.5mm
- Q1, Q2: value (none) -> AO3407; footprint (none) -> Package_TO_SOT_SMD:SOT-23
- R1, R3: value (none) -> 5.1k; footprint (none) -> Resistor_SMD:R_0603_1608Metric
- R10: value (none) -> 2.3k; footprint (none) -> Resistor_SMD:R_0603_1608Metric
- R2, R5: value (none) -> 2M; footprint (none) -> Resistor_SMD:R_0603_1608Metric
- R4, R9: value (none) -> 1K; footprint (none) -> Resistor_SMD:R_0603_1608Metric
- R6: value (none) -> 100k; footprint (none) -> Resistor_SMD:R_0603_1608Metric
- R7: value (none) -> 100K; footprint (none) -> Resistor_SMD:R_0603_1608Metric
- R8: value (none) -> 10M; footprint (none) -> Resistor_SMD:R_0603_1608Metric
- SW46: value (none) -> RST
- U2: value (none) -> MIC5219-3.3YM5; footprint (none) -> Library:SOT-23-5
- U3: value (none) -> USBLC6-2SC6; footprint (none) -> Library:SOT-23-6
- U4: value (none) -> E73-2G4M08S1C; footprint kien242:E73-2G4M08S1C -> kien242:E73-2G4M08S1C-kien242
- U5: value (none) -> TP4054; footprint (none) -> Library:SOT-23-5
Connections:
- net +3V3: now also U4.19 (VDD), U4.23 (VDDH)
- net GND: now also U4.21 (GND), U4.24 (GND), U4.5 (GND)

Commit message: Update
Parts:
- removed D43: BLUE, LED_SMD:LED_0603_1608Metric, symbol Device:LED
- removed R4: 1K, Resistor_SMD:R_0603_1608Metric, symbol Device:R_Small
- added Y1: 32.768kHz, Library:Crystal_0603, symbol Device:Crystal_Small
- U2, U5: footprint Library:SOT-23-5 -> Package_TO_SOT_SMD:SOT-23-5
- U3: footprint Library:SOT-23-6 -> Package_TO_SOT_SMD:SOT-23-6
- renumbered D44 to D43, D45 to D44, R5 to R4, R6 to R5, R7 to R6, R8 to R7, R9 to R8, R10 to R9
Connections:
- net +5V: now also U4.27 (VBUS)
- net BATTERY_PIN: now also U4.3 (P0.03/AIN1)
- net D+: now also U3.1 (I/O1), U4.31 (D+); no longer U3.3 (I/O2)
- net D-: now also U3.3 (I/O2), U4.29 (D-); no longer U3.1 (I/O1)
- net DP+: now also U3.6 (I/O1); no longer U3.4 (I/O2)
- net DP-: now also U3.4 (I/O2); no longer U3.6 (I/O1)
- net RST: now also U4.26 (P0.18/RESET), U4.6 (P1.13)
- net SWCLK: now also U4.39 (SWDCLK)
- net SWDIO: now also U4.37 (SWDIO)
- net VBAT: no longer U5.3 (VBAT)
- net at U4.11 (P0.00/XL1): now also Y1.1
- net at U4.13 (P0.01/XL2): now also Y1.2
- net SCL: now reaches U4.33 (P0.13)
- net SDA: now reaches U4.35 (P0.24)
- net TX: now reaches U4.41 (P0.09/NFC1)
- net RX: now reaches U4.43 (P0.10/NFC2)
- net +3V3 renamed nRF_VDD
- new net VBAT_CHG: U5.3 (VBAT)

Commit message: Update PCB
Connections:
- net POWER_PIN: now also U4.9 (P0.31/AIN7)
- net col2: now reaches U4.10 (P0.30/AIN6)
- net col3: now reaches U4.12 (P0.26)
- net col4: now reaches U4.14 (P0.06)
- net col5: now reaches U4.15 (P0.05/AIN3)
- net RGB_BLACKPILL: now reaches U4.16 (P0.08)
- net row0: now reaches U4.17 (P1.09)
- net row1: now reaches U4.18 (P0.04/AIN2)
- net col1': now reaches U4.20 (P0.12)
- net col2': now reaches U4.22 (P0.07)
- net col3': now reaches U4.28 (P0.15)
- net col0: now reaches U4.30 (P0.17)
- net col1: now reaches U4.32 (P0.20)
- net row2: now reaches U4.34 (P0.22)
- net row3: now reaches U4.36 (P1.00)
- net row4: now reaches U4.38 (P1.02)
- net ENCA: now reaches U4.40 (P1.04)
- net ENCB: now reaches U4.42 (P1.06)
