File: PCB/PCB/v1.1/RGB.kicad_sch (KiCad schematic)
At the start: 36 parts

Commit message: update PCB file
Parts:
- C1, C10, C11, C12, C13, C14, C15, C16, C17, C18, C19, C2, C20, C3, C4, C5, C6, C7, C8, C9: renamed from U; value (none) -> 104; footprint (none) -> Capacitor_SMD:C_0603_1608Metric
- J26, J27, J28, J29: renamed from U; value (none) -> (none); footprint (none) -> Library:Conn_01x01
- JP10: renamed from U; value (none) -> Jump LED; footprint (none) -> Jumper:SolderJumper-2_P1.3mm_Open_Pad1.0x1.5mm
- JP9: renamed from U; value (none) -> Jump LED; footprint (none) -> Jumper:SolderJumper-2_P1.3mm_Open_RoundedPad1.0x1.5mm
- LED1, LED10, LED2, LED3, LED4, LED5, LED6, LED7, LED8, LED9: renamed from U; value (none) -> 6812; footprint (none) -> kien242:SK6812MINI-FLIP

Commit message: update PCB file
Connections:
- net +3V3 renamed VCC
